Commit message: NAV2 Commit - Desenvolvimento inicial da navegação autônoma
Co-authored-by: Giovane-F-Moreira <64364499+Giovane-F-Moreira@users.noreply.github.com>

File: nara-sim/src/smartwheelchair/urdf/narawheelchair.xacro (robot description, xacro)
@@ -164,5 +164,5 @@
 </link>
 <joint name="robot_footprint_joint" type="fixed">
-  <origin xyz="0 0 0" rpy="0 0 0" />
+  <origin xyz="0.25395 0 0" rpy="0 0 0" />
   <parent link="robot_footprint"/>
   <child link="base_link" />

Commit message: Recolocação do Lidar no 3D na cadeira

File: nara-sim/src/smartwheelchair/urdf/narawheelchair.xacro (robot description, xacro)
@@ -172,5 +172,5 @@
 <joint name="hokuyo_joint" type="fixed">
   <axis xyz="0 1 0" />
-  <origin xyz="0.59 0.0 0.265" rpy="0 3.14 3.14" />
+  <origin xyz="0.59 0.0 0.065" rpy="0 3.14 3.14" />
   <parent link="base_link"/>
   <child link="hokuyo_link"/>
