File: nara-main/Circuito/Projeto da Placa PCB no KiCad/placa_nara.kicad_pcb (KiCad board)
At the start: 2 copper layers, 49 x 26 mm, 8 parts, among them J1 JETSON, J2 Motor Right, J3 Motor Left, J4 Encoder Right, J5 Encoder Left, U2 module_mpu6050, U3 LLC Encoders

Commit message: Projeto da Placa PCB Atualizado
Parts:
- removed J2: Motor Right, Connector_PinSocket_1.00mm:PinSocket_1x06_P1.00mm_Vertical
- removed J3: Motor Left, Connector_PinSocket_1.00mm:PinSocket_1x06_P1.00mm_Vertical
- removed J4: Encoder Right, Connector_PinSocket_1.00mm:PinSocket_1x04_P1.00mm_Vertical
- removed J5: Encoder Left, Connector_PinSocket_1.00mm:PinSocket_1x04_P1.00mm_Vertical
- added ENCODER_LEFT1: Conn_01x04_Pin, Connector_PinHeader_2.54mm:PinHeader_1x04_P2.54mm_Vertical, F.Cu at (67.5, 149.5)
- added ENCODER_RIGHT1: Conn_01x04_Pin, Connector_PinHeader_2.54mm:PinHeader_1x04_P2.54mm_Vertical, F.Cu at (127.0, 149.5)
- added JETSON1: Conn_01x02_Pin, Connector_PinHeader_2.54mm:PinHeader_1x02_P2.54mm_Vertical, F.Cu at (66.5, 95.5)
- added MOTOR_LEFT1: Conn_01x06_Pin, Connector_PinHeader_2.54mm:PinHeader_1x06_P2.54mm_Vertical, F.Cu at (88.0, 77.0)
- added MOTOR_RIGHT1: Conn_01x06_Pin, Connector_PinHeader_2.54mm:PinHeader_1x06_P2.54mm_Vertical, F.Cu at (111.5, 77.0)
- added REF**: MountingHole_3.2mm_M3, MountingHole:MountingHole_3.2mm_M3, F.Cu at (151.5, 162.5)
- added REF**: MountingHole_3.2mm_M3, MountingHole:MountingHole_3.2mm_M3, F.Cu at (46.5, 58.5)
- added REF**: MountingHole_3.2mm_M3, MountingHole:MountingHole_3.2mm_M3, F.Cu at (151.5, 58.5)
- added REF**: MountingHole_3.2mm_M3, MountingHole:MountingHole_3.2mm_M3, F.Cu at (46.5, 162.5)
- added SENSOR_TENSAO1: Conn_01x02_Pin, Connector_PinHeader_2.54mm:PinHeader_1x02_P2.54mm_Vertical, F.Cu at (78.5, 130.2)
- J1: value JETSON -> Screw_Terminal_01x02; footprint TerminalBlock_Phoenix:TerminalBlock_Phoenix_MKDS-1,5-2_1x02_P5.00mm_Horizontal -> TerminalBlock_Phoenix:TerminalBlock_Phoenix_MKDS-1,5-2-5.08_1x02_P5.08mm_Horizontal
- U2: value module_mpu6050 -> LLC_4CH_I2C; footprint usini_sensors:module_mpu6050 -> LLC_4CH_I2C:LLC_4CH_I2C_MODULE
- U3: value LLC Encoders -> module_mpu6050; footprint LLC_4CH_I2C:LLC_4CH_I2C_MODULE -> usini_sensors:module_mpu6050
- moved U2 82.8 mm to (72.3, 112.8), turned to 0 degrees
- moved U1 73.2 mm to (98.9, 117.5), turned to 0 degrees
- moved U3 61.1 mm to (121.5, 123.5), turned to 0 degrees
- moved J1 46.3 mm to (131.5, 136.5), turned to 90 degrees
Connections:
- J1 pad 1: /VCC_5V -> GND
- J1 pad 2: /GND_Jetson -> /3.3V
- U1 pad 10: /ENCODER_LEFT_A_LV -> /ENCODER_LEFT_B_LV
- U1 pad 17: /GND_Jetson -> GND
- U1 pad 24: unconnected-(U1-GPIO18-Pad24) -> /BATTERY_VOLTAGE_2
- U1 pad 26: Net-(U1-GPIO21) -> /IMU_SDA
- U1 pad 29: Net-(U1-GPIO22) -> /IMU_SCL
- U1 pad 3: unconnected-(U1-GPIO13-Pad3) -> /BATTERY_VOLTAGE_1
- U1 pad 30: /Motor ENABLE -> /MOTOR_ENABLE
- U1 pad 5: /Motor Right R_PWM -> /MOTOR_RIGHT_RPWM
- U1 pad 6: /Motor Right L_PWM -> /MOTOR_RIGHT_LPWM
- U1 pad 7: /Motor Left L_PWM -> /MOTOR_LEFT_LPWM
- U1 pad 8: /Motor Left R_PWM -> /MOTOR_LEFT_RPWM
- U1 pad 9: /ENCODER_LEFT_B_LV -> /ENCODER_LEFT_A_LV
- U2 pad 1: /3.3V -> /ENCODER_RIGHT_A_HV
- U2 pad 2: /GND_Jetson -> /ENCODER_RIGHT_B_HV
- U2 pad 3: Net-(U1-GPIO22) -> /5V
- U2 pad 4: Net-(U1-GPIO21) -> GND
- U2 pad 5: unconnected-(U2-XDA-Pad5) -> /ENCODER_LEFT_A_HV
- U2 pad 6: unconnected-(U2-XCL-Pad6) -> /ENCODER_LEFT_B_HV
- U2 pad 7: unconnected-(U2-ADD-Pad7) -> /ENCODER_RIGHT_A_LV
- U2 pad 8: unconnected-(U2-INT-Pad8) -> /ENCODER_RIGHT_B_LV
- U3 pad 1: Net-(J4-Pin_1) -> /3.3V
- U3 pad 2: Net-(J4-Pin_2) -> GND
- U3 pad 3: /VCC_5V -> /IMU_SCL
- U3 pad 4: /GND_Jetson -> /IMU_SDA
- U3 pad 5: Net-(J4-Pin_2) -> unconnected-(U3-XDA-Pad5)
- U3 pad 6: Net-(J5-Pin_2) -> unconnected-(U3-XCL-Pad6)
- U3 pad 7: /ENCODER_RIGHT_A_LV -> unconnected-(U3-ADD-Pad7)
- U3 pad 8: /ENCODER_RIGHT_B_LV -> unconnected-(U3-INT-Pad8)
Routing:
- net GND: track 0.00 -> 179.5 mm
- net /5V: track 0.00 -> 121.3 mm
- net /ENCODER_RIGHT_A_LV: track 121.9 -> 9.55 mm
- net /3.3V: track 66.1 -> 177.4 mm
- net /ENCODER_RIGHT_B_HV: track 0.00 -> 109.2 mm
- net /ENCODER_RIGHT_A_HV: track 0.00 -> 100.1 mm
- net /GND_Jetson: track 88.6 -> 0.00 mm
- net /MOTOR_ENABLE: track 0.00 -> 79.8 mm
- net /VCC_5V: track 68.2 -> 0.00 mm
- net /MOTOR_RIGHT_RPWM: track 0.00 -> 63.0 mm
- net /MOTOR_RIGHT_LPWM: track 0.00 -> 59.3 mm
- net /MOTOR_LEFT_LPWM: track 0.00 -> 49.3 mm
- net /MOTOR_LEFT_RPWM: track 0.00 -> 46.1 mm
- net /BATTERY_VOLTAGE_2: track 0.00 -> 44.4 mm
- net /ENCODER_LEFT_A_HV: track 0.00 -> 42.6 mm
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- added copper zone on B.Cu, net GND
Other:
- board size 49 x 26 mm -> 115 x 112 mm
- board text added: "NOBLENARA 2026.2"

Commit message: Atualizado o projeto da placa pcb correspondente ao modelo físico
Parts:
- moved REF** 9.12 mm to (55.5, 161.0)
- moved REF** 8.63 mm to (55.0, 60.0)
- moved REF** 5.70 mm to (146.0, 161.0)
- moved REF** 5.22 mm to (146.5, 60.0)
Routing:
- net GND: track 179.5 -> 128.1 mm, vias 0 -> 4
- net /ENCODER_LEFT_A_LV: track 18.3 -> 21.8 mm
- net /ENCODER_RIGHT_B_HV: track 109.2 -> 112.0 mm
- net /5V: track 121.3 -> 123.1 mm
- net /3.3V: track 177.4 -> 178.5 mm
- net /MOTOR_RIGHT_RPWM: track 63.0 -> 63.6 mm
Other:
- board size 115 x 112 mm -> 102 x 112 mm
- board text added: "3.3V"
- board text added: "5V"
- board text added: "A"
- board text added: "ADD"
- board text added: "B"
- board text added: "CONVERSOR DE NÍVEL LÓGICO"
- board text added: "DAVID MANHÃES; PEDRO PAULO; PEDRO AUGUSTO; FABRÍCIA ASTRID; CAIO ANDRADE"
- board text added: "ENABLE"
- board text added: "ENCODER LEFT"
- board text added: "ENCODER RIGHT"
- board text added: "ESP32"
- board text added: "GND"
- board text added: "HV"
- board text added: "HV1"
- board text added: "HV2"
- board text added: "HV3"
- board text added: "HV4"
- board text added: "IMU"
- board text added: "INT"
- board text added: "JETSON"
- board text added: "LV"
- board text added: "LV1"
- board text added: "LV2"
- board text added: "LV3"
- board text added: "LV4"
- board text added: "L_PWM"
- board text added: "MOTOR LEFT"
- board text added: "MOTOR RIGHT"
- board text added: "R_PWM"
- board text added: "SCL"
- board text added: "SDA"
- board text added: "SENSOR DE TENSÃO"
- board text added: "USB"
- board text added: "V1"
- board text added: "V2"
- board text added: "VCC"
- board text added: "XCL"
- board text added: "XDA"
